File: PowerAdjustmentMonitor.sch (KiCad schematic (older format))
At the start: 15 parts, among them U10 LM317, U11 LM317, U8 7805, U9 7805

Commit message: Associating The Power Modify Module
Parts:
- removed JP2, JP3: JUMPER, ~, symbol JUMPER
- removed U10: LM317, ~, symbol LM317
- removed U8, U9: 7805, ~, symbol 7805
- added C14, C15, C16, C17, C18, C19, C20, C21, C22, C23, C24, C25: C, ~, symbol C
- added D10, D3, D6, D7, D8, D9: DIODE, ~, symbol DIODE
- added R52, R53, R54, R55: R, ~, symbol R
- added U6, U8: LM337T, TO-220, symbol LM337T
- added U9: LM317, ~, symbol LM317
Connections:
- net labels removed: V-_MON
- wire segments 57 -> 96
Other:
- note added: "-1.5V to -10 V Output"
- note added: "-10V Output\n"
- note added: "1.5 to 10 V Output"
- note added: "10V Output\n"
- moved on the sheet: JP1, R20, R21, U11

Commit message: Placing the Power Modify Module
Parts:
- added D11, D12: MMBD914-7-F, ~, symbol DIODE
- D10, D3, D6, D7, D8, D9: value DIODE -> MMBD914-7-F
- R18, R21: value R -> 715
- R19, R20: value RVAR -> 5K
Connections:
- net +12V: now also D9.2 (K); no longer D3.2 (K)
- net -12V: now also D3.2 (K), D7.2 (K)
- net AGND: now also R55.1, D12.2 (K)
- net FE_V+: now also D9.1 (A); no longer D6.1 (A)
- net FE_V-: now also D7.1 (A); no longer D9.2 (K)
- net V+_ADJ: now also D6.1 (A); no longer D3.1 (A)
- net V-_ADJ: now also D3.1 (A), D11.1 (A); no longer D7.2 (K)
- net at C21.2, R52.2, R53.1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: now also D12.1 (A); no longer D9.1 (A)
- net at C18.1, R18.1, R19.1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: now also D11.2 (K); no longer D7.1 (A)
