File: PowerAdjustmentMonitor.sch (KiCad schematic (older format))
At the start: 37 parts, among them U11 LM317, U6 LM337T, U8 LM337T, U9 LM317

Commit message: Layout Work Session 4 Output
Parts:
- removed JP1: JUMPER, ~, symbol JUMPER
Connections:
- net labels added: GND_PWR, GND_TC
- net labels removed: AGND, GND
- wire segments 105 -> 103
Other:
- moved on the sheet: C14, C15, C16, C17, C18, C19, C20, C21, C22, C23, C24, C25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

Commit message: Layout Work Session 5
Connections:
- net labels added: AGND
- net labels removed: GND_TC
Changed lines of the file:
@@
-EESchema Schematic File Version 2  date 11/7/2013 10:50:27 PM
+EESchema Schematic File Version 2  date 11/9/2013 9:10:12 PM
 LIBS:power
 LIBS:device
@@
 Sheet 5 9
 Title ""
-Date "8 nov 2013"
+Date "10 nov 2013"
 Rev ""
 Comp ""
@@
 $EndComp
 $Comp
-L FE_V+ #PWR028
+L FE_V+ #PWR025
 U 1 1 523E0975
 P 4950 1800
-F 0 "#PWR028" H 4950 1900 30  0001 C CNN
+F 0 "#PWR025" H 4950 1900 30  0001 C CNN
 F 1 "FE_V+" H 4950 1900 30  0000 C CNN
 F 2 "~" H 4950 1800 60  0000 C CNN
@@
 Connection ~ 3750 3150
 $Comp
-L GND_PWR #PWR?
+L GND_PWR #PWR026
 U 1 1 527CFD60
 P 6550 3900
-F 0 "#PWR?" H 6550 3900 30  0001 C CNN
+F 0 "#PWR026" H 6550 3900 30  0001 C CNN
 F 1 "GND_PWR" H 6550 3830 30  0000 C CNN
 F 2 "~" H 6550 3900 60  0000 C CNN
@@
 $EndComp
 $Comp
-L GND_PWR #PWR?
-U 1 1 527CFD76
-P 3150 5200
-F 0 "#PWR?" H 3150 5200 30  0001 C CNN
-F 1 "GND_PWR" H 3150 5130 30  0000 C CNN
-F 2 "~" H 3150 5200 60  0000 C CNN
-F 3 "~" H 3150 5200 60  0000 C CNN
-	1    3150 5200
-	-1   0    0    1
-$EndComp
-$Comp
-L -12V #PWR?
+L -12V #PWR027
 U 1 1 527CFD7C
 P 5950 5250
-F 0 "#PWR?" H 5950 5380 20  0001 C CNN
+F 0 "#PWR027" H 5950 5380 20  0001 C CNN
 F 1 "-12V" H 5950 5350 30  0000 C CNN
 F 2 "" H 5950 5250 60  0000 C CNN
@@
 	1550 4050 1550 4700
 $Comp
-L +12V #PWR?
+L +12V #PWR028
 U 1 1 527CFEC0
 P 1500 1700
-F 0 "#PWR?" H 1500 1650 20  0001 C CNN
+F 0 "#PWR028" H 1500 1650 20  0001 C CNN
 F 1 "+12V" H 1500 1800 30  0000 C CNN
 F 2 "" H 1500 1700 60  0000 C CNN
@@
 Wire Wire Line
 	6400 1850 6400 1700
-$Comp
-L GND_TC #PWR?
-U 1 1 527D00A8
-P 1250 3350
-F 0 "#PWR?" H 1250 3350 30  0001 C CNN
-F 1 "GND_TC" H 1250 3280 30  0000 C CNN
-F 2 "~" H 1250 3350 60  0000 C CNN
-F 3 "~" H 1250 3350 60  0000 C CNN
-	1    1250 3350
-	1    0    0    -1
-$EndComp
 Wire Wire Line
 	1250 3150 4200 3150
@@
 	6550 3900 6550 3800
 Connection ~ 6800 3800
+$Comp
+L AGND #PWR029
+U 1 1 527EFACA
+P 1250 3350
+F 0 "#PWR029" H 1250 3350 40  0001 C CNN
+F 1 "AGND" H 1250 3280 50  0000 C CNN
+F 2 "~" H 1250 3350 60  0000 C CNN
+F 3 "~" H 1250 3350 60  0000 C CNN
+	1    1250 3350
+	1    0    0    -1
+$EndComp
 $EndSCHEMATC
