File: Thermocouple.sch (KiCad schematic (older format))
At the start: 22 parts, among them P2 CONN_3X2, P3 CONN_2, U2 MCP3901, U3 LMT84, U4 OPA4170

Commit message: Layout Work Session 5
Connections:
- net GND_TC renamed AGND
Changed lines of the file:
@@
-EESchema Schematic File Version 2  date 11/7/2013 10:50:27 PM
+EESchema Schematic File Version 2  date 11/9/2013 9:10:12 PM
 LIBS:power
 LIBS:device
@@
 Sheet 2 9
 Title ""
-Date "8 nov 2013"
+Date "10 nov 2013"
 Rev ""
 Comp ""
@@
 Connection ~ 4800 6800
 $Comp
-L +5V #PWR03
+L +5V #PWR01
 U 1 1 5257A1D1
 P 5600 5000
-F 0 "#PWR03" H 5600 5090 20  0001 C CNN
+F 0 "#PWR01" H 5600 5090 20  0001 C CNN
 F 1 "+5V" H 5600 5090 30  0000 C CNN
 F 2 "~" H 5600 5000 60  0000 C CNN
@@
 	6050 3800 6250 3800
 $Comp
-L +5V #PWR06
+L +5V #PWR02
 U 1 1 5257A5A4
 P 5600 5000
-F 0 "#PWR06" H 5600 5090 20  0001 C CNN
+F 0 "#PWR02" H 5600 5090 20  0001 C CNN
 F 1 "+5V" H 5600 5090 30  0000 C CNN
 F 2 "~" H 5600 5000 60  0000 C CNN
@@
 $EndComp
 $Comp
-L +5V #PWR07
+L +5V #PWR03
 U 1 1 5257A5AA
 P 3100 1300
-F 0 "#PWR07" H 3100 1390 20  0001 C CNN
+F 0 "#PWR03" H 3100 1390 20  0001 C CNN
 F 1 "+5V" H 3100 1390 30  0000 C CNN
 F 2 "~" H 3100 1300 60  0000 C CNN
@@
 	3100 4600 3100 4850
 $Comp
-L +5V #PWR012
+L +5V #PWR04
 U 1 1 5257AAC2
 P 2400 1300
-F 0 "#PWR012" H 2400 1390 20  0001 C CNN
+F 0 "#PWR04" H 2400 1390 20  0001 C CNN
 F 1 "+5V" H 2400 1390 30  0000 C CNN
 F 2 "~" H 2400 1300 60  0000 C CNN
@@
 $EndComp
 $Comp
-L FE_V+ #PWR013
+L FE_V+ #PWR05
 U 1 1 526E01E1
 P 6250 3850
-F 0 "#PWR013" H 6250 3950 30  0001 C CNN
+F 0 "#PWR05" H 6250 3950 30  0001 C CNN
 F 1 "FE_V+" H 6250 3950 30  0000 C CNN
 F 2 "~" H 6250 3850 60  0000 C CNN
@@
 $EndComp
 $Comp
-L FE_V+ #PWR014
+L FE_V+ #PWR06
 U 1 1 526E01F1
 P 9000 5000
-F 0 "#PWR014" H 9000 5100 30  0001 C CNN
+F 0 "#PWR06" H 9000 5100 30  0001 C CNN
 F 1 "FE_V+" H 9000 5100 30  0000 C CNN
 F 2 "~" H 9000 5000 60  0000 C CNN
@@
 $EndComp
 $Comp
-L FE_V+ #PWR015
+L FE_V+ #PWR07
 U 1 1 526E020D
 P 9000 2850
-F 0 "#PWR015" H 9000 2950 30  0001 C CNN
+F 0 "#PWR07" H 9000 2950 30  0001 C CNN
 F 1 "FE_V+" H 9000 2950 30  0000 C CNN
 F 2 "~" H 9000 2850 60  0000 C CNN
@@
 $EndComp
 $Comp
-L GND_TC #PWR?
-U 1 1 527CE7CA
+L AGND #PWR08
+U 1 1 527EEF67
+P 3100 4850
+F 0 "#PWR08" H 3100 4850 40  0001 C CNN
+F 1 "AGND" H 3100 4780 50  0000 C CNN
+F 2 "~" H 3100 4850 60  0000 C CNN
+F 3 "~" H 3100 4850 60  0000 C CNN
+	1    3100 4850
+	1    0    0    -1
+$EndComp
+$Comp
+L AGND #PWR09
+U 1 1 527EEF6D
+P 2300 4850
+F 0 "#PWR09" H 2300 4850 40  0001 C CNN
+F 1 "AGND" H 2300 4780 50  0000 C CNN
+F 2 "~" H 2300 4850 60  0000 C CNN
+F 3 "~" H 2300 4850 60  0000 C CNN
+	1    2300 4850
+	1    0    0    -1
+$EndComp
+$Comp
+L AGND #PWR010
+U 1 1 527EEF73
+P 1750 1650
+F 0 "#PWR010" H 1750 1650 40  0001 C CNN
+F 1 "AGND" H 1750 1580 50  0000 C CNN
+F 2 "~" H 1750 1650 60  0000 C CNN
+F 3 "~" H 1750 1650 60  0000 C CNN
+	1    1750 1650
+	1    0    0    -1
+$EndComp
+$Comp
+L AGND #PWR011
+U 1 1 527EEF79
+P 3700 1600
+F 0 "#PWR011" H 3700 1600 40  0001 C CNN
+F 1 "AGND" H 3700 1530 50  0000 C CNN
+F 2 "~" H 3700 1600 60  0000 C CNN
+F 3 "~" H 3700 1600 60  0000 C CNN
+	1    3700 1600
+	1    0    0    -1
+$EndComp
+$Comp
+L AGND #PWR012
+U 1 1 527EEF7F
+P 5600 2800
+F 0 "#PWR012" H 5600 2800 40  0001 C CNN
+F 1 "AGND" H 5600 2730 50  0000 C CNN
+F 2 "~" H 5600 2800 60  0000 C CNN
+F 3 "~" H 5600 2800 60  0000 C CNN
+	1    5600 2800
+	1    0    0    -1
+$EndComp
+$Comp
+L AGND #PWR013
+U 1 1 527EEF85
+P 5550 4000
+F 0 "#PWR013" H 5550 4000 40  0001 C CNN
+F 1 "AGND" H 5550 3930 50  0000 C CNN
+F 2 "~" H 5550 4000 60  0000 C CNN
+F 3 "~" H 5550 4000 60  0000 C CNN
+	1    5550 4000
+	1    0    0    -1
+$EndComp
+$Comp
+L AGND #PWR014
+U 1 1 527EEF8B
+P 4900 4700
+F 0 "#PWR014" H 4900 4700 40  0001 C CNN
+F 1 "AGND" H 4900 4630 50  0000 C CNN
+F 2 "~" H 4900 4700 60  0000 C CNN
+F 3 "~" H 4900 4700 60  0000 C CNN
+	1    4900 4700
+	1    0    0    -1
+$EndComp
+$Comp
+L AGND #PWR015
+U 1 1 527EEF91
 P 4800 6900
-F 0 "#PWR?" H 4800 6900 30  0001 C CNN
-F 1 "GND_TC" H 4800 6830 30  0000 C CNN
+F 0 "#PWR015" H 4800 6900 40  0001 C CNN
+F 1 "AGND" H 4800 6830 50  0000 C CNN
 F 2 "~" H 4800 6900 60  0000 C CNN
 F 3 "~" H 4800 6900 60  0000 C CNN
@@
 	1    0    0    -1
 $EndComp
-$Comp
-L GND_TC #PWR?
-U 1 1 527CE7D0
-P 3100 4850
-F 0 "#PWR?" H 3100 4850 30  0001 C CNN
-F 1 "GND_TC" H 3100 4780 30  0000 C CNN
-F 2 "~" H 3100 4850 60  0000 C CNN
-F 3 "~" H 3100 4850 60  0000 C CNN
-	1    3100 4850
-	1    0    0    -1
-$EndComp
-$Comp
-L GND_TC #PWR?
-U 1 1 527CE7D6
-P 2300 4850
-F 0 "#PWR?" H 2300 4850 30  0001 C CNN
-F 1 "GND_TC" H 2300 4780 30  0000 C CNN
-F 2 "~" H 2300 4850 60  0000 C CNN
-F 3 "~" H 2300 4850 60  0000 C CNN
-	1    2300 4850
-	1    0    0    -1
-$EndComp
-$Comp
-L GND_TC #PWR?
-U 1 1 527CE7DC
-P 1750 1650
-F 0 "#PWR?" H 1750 1650 30  0001 C CNN
-F 1 "GND_TC" H 1750 1580 30  0000 C CNN
-F 2 "~" H 1750 1650 60  0000 C CNN
-F 3 "~" H 1750 1650 60  0000 C CNN
-	1    1750 1650
-	1    0    0    -1
-$EndComp
-$Comp
-L GND_TC #PWR?
-U 1 1 527CE7E2
-P 3700 1600
-F 0 "#PWR?" H 3700 1600 30  0001 C CNN
-F 1 "GND_TC" H 3700 1530 30  0000 C CNN
-F 2 "~" H 3700 1600 60  0000 C CNN
-F 3 "~" H 3700 1600 60  0000 C CNN
-	1    3700 1600
-	1    0    0    -1
-$EndComp
-$Comp
-L GND_TC #PWR?
-U 1 1 527CE7E8
-P 5600 2800
-F 0 "#PWR?" H 5600 2800 30  0001 C CNN
-F 1 "GND_TC" H 5600 2730 30  0000 C CNN
-F 2 "~" H 5600 2800 60  0000 C CNN
-F 3 "~" H 5600 2800 60  0000 C CNN
-	1    5600 2800
-	1    0    0    -1
-$EndComp
-$Comp
-L GND_TC #PWR?
-U 1 1 527CE7EE
-P 5550 4000
-F 0 "#PWR?" H 5550 4000 30  0001 C CNN
-F 1 "GND_TC" H 5550 3930 30  0000 C CNN
-F 2 "~" H 5550 4000 60  0000 C CNN
-F 3 "~" H 5550 4000 60  0000 C CNN
-	1    5550 4000
-	1    0    0    -1
-$EndComp
-$Comp
-L GND_TC #PWR?
-U 1 1 527CE7F4
-P 4900 4700
-F 0 "#PWR?" H 4900 4700 30  0001 C CNN
-F 1 "GND_TC" H 4900 4630 30  0000 C CNN
-F 2 "~" H 4900 4700 60  0000 C CNN
-F 3 "~" H 4900 4700 60  0000 C CNN
-	1    4900 4700
-	1    0    0    -1
-$EndComp
