File: BenchBuddy.kicad_pcb (KiCad board)
At the start: 4 copper layers, 165.1 x 63.5 mm, 130 parts, among them K1 1461069-5, P1 24 Pin MiniFit JR, P2 CONN_3X2, P3 CONN_2, P4 12 Pin Terminal Block, P5 3 Pin TB, Q1 2N3904, Q2 DMN65D8L-7, Q3 AOD476, Q4 AOD476, SW1 Power Switch, U1 LTV-816S, U11 LM317, U2 MCP3901, U3 LMT84, U4 OPA4170, U5 MCP4801, U6 LM337T, U7 AP5726, U8 LM337T, U9 LM317

Commit message: Layout Work Session 6 Output
Parts:
- added JP2: JUMPER, PIN_ARRAY_2X1, F.Cu at (87.6, 108.8)
- added JP3: JUMPER, PIN_ARRAY_2X1, F.Cu at (94.6, 115.5)
- added JP4: JUMPER, PIN_ARRAY_2X1, F.Cu at (87.6, 119.2)
- C11, C9, D10, D11, D12, D3, D6, D7, D8, D9, Q2, R48, R49: moved to B.Cu
- C25, R12, R15, R18, R21, R24, R25, R44, R45, R52, R54: moved to F.Cu
- moved JP1 129.9 mm to (94.7, 111.4)
- moved R25 111.4 mm to (148.8, 94.2), turned to 270 degrees
- moved R21 111.4 mm to (140.7, 80.8), turned to 0 degrees
- moved R22 102.4 mm to (151.3, 94.1), turned to 90 degrees
- moved R23 101.5 mm to (149.2, 94.3)
- moved R24 98.0 mm to (151.3, 94.2), turned to 90 degrees
- moved R18 93.1 mm to (140.7, 83.5)
- moved C18 86.0 mm to (161.4, 89.5)
- moved D3 83.7 mm to (156.4, 83.0), turned to 90 degrees
- moved D11 82.7 mm to (160.7, 83.1), turned to 180 degrees
- moved C16 75.9 mm to (152.5, 85.3), turned to 90 degrees
- moved C19 72.0 mm to (174.8, 92.0), turned to 0 degrees
- moved C23 71.4 mm to (157.0, 89.4), turned to 180 degrees
- moved C13 71.3 mm to (184.0, 114.4), turned to 0 degrees
- moved R15 71.2 mm to (168.2, 112.4)
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Connections:
- JP1 pad 1: AGND -> GND
- JP1 pad 2: GND -> AGND
- P4 pad 8: GND_PWR -> +5V
- P4 pad 9: +5V -> GND_PWR
Routing:
- net +3.3V: track 0.00 -> 145.5 mm
- net N-00000107: track 0.00 -> 50.3 mm
- net +12P: track 2.27 -> 48.7 mm, vias 1 -> 2
- net GND: track 0.00 -> 32.1 mm
- net -12P: track 0.00 -> 31.6 mm, vias 0 -> 1
- net N-00000102: track 0.00 -> 19.8 mm
- net +5P: track 2.70 -> 10.5 mm, vias 1 -> 2
- net +5V: track 1.78 -> 7.83 mm, vias 1 -> 2
- net -12V: track 199.9 -> 205.8 mm
- net N-00000103: track 0.00 -> 5.80 mm
- net +12C: vias 2 -> 1
- net /Fan/FAN_OUT-: vias 0 -> 1
- added copper zone on GND, net GND
