File: Fan.sch (KiCad schematic (older format))
At the start: 11 parts, among them Q2 DMN65D8L-7, Q3 AOD476, Q4 AOD476, U4 OPA4170, U5 MCP4801

Commit message: Layout Work Session 4 Output
Connections:
- net labels added: GND_FAN
- net labels removed: AGND, GND
Changed lines of the file:
@@
-EESchema Schematic File Version 2  date 11/2/2013 7:04:39 PM
+EESchema Schematic File Version 2  date 11/7/2013 10:50:27 PM
 LIBS:power
 LIBS:device
@@
 Sheet 6 9
 Title ""
-Date "2 nov 2013"
+Date "8 nov 2013"
 Rev ""
 Comp ""
@@
 	1    0    0    -1
 $EndComp
-$Comp
-L AGND #PWR41
-U 1 1 523698EE
-P 4700 3750
-F 0 "#PWR41" H 4700 3750 40  0001 C CNN
-F 1 "AGND" H 4700 3680 50  0000 C CNN
-F 2 "" H 4700 3750 60  0000 C CNN
-F 3 "" H 4700 3750 60  0000 C CNN
-	1    4700 3750
-	1    0    0    -1
-$EndComp
 Text HLabel 1450 4500 0    60   Output ~ 0
 CURR_MEAS
@@
 FAN_MODE
 $Comp
-L +12C #PWR44
+L +12C #PWR034
 U 1 1 5243907A
 P 7900 1000
-F 0 "#PWR44" H 7900 970 30  0001 C CNN
+F 0 "#PWR034" H 7900 970 30  0001 C CNN
 F 1 "+12C" H 7900 1110 40  0000 C CNN
 F 2 "~" H 7900 1000 60  0000 C CNN
@@
 	2000 1950 1900 1950
 Connection ~ 2000 1950
-$Comp
-L AGND #PWR38
-U 1 1 525C14F8
-P 1350 2050
-F 0 "#PWR38" H 1350 2050 40  0001 C CNN
-F 1 "AGND" H 1350 1980 50  0000 C CNN
-F 2 "" H 1350 2050 60  0000 C CNN
-F 3 "" H 1350 2050 60  0000 C CNN
-	1    1350 2050
-	1    0    0    -1
-$EndComp
 Wire Wire Line
 	1350 2050 1350 1950
@@
 	1350 1950 1500 1950
 $Comp
-L +5V #PWR39
+L +5V #PWR036
 U 1 1 525C1500
 P 2000 1700
-F 0 "#PWR39" H 2000 1790 20  0001 C CNN
+F 0 "#PWR036" H 2000 1790 20  0001 C CNN
 F 1 "+5V" H 2000 1790 30  0000 C CNN
 F 2 "~" H 2000 1700 60  0000 C CNN
 F 3 "~" H 2000 1700 60  0000 C CNN
 	1    2000 1700
-	1    0    0    -1
-$EndComp
-$Comp
-L AGND #PWR40
-U 1 1 525C1506
-P 2000 3950
-F 0 "#PWR40" H 2000 3950 40  0001 C CNN
-F 1 "AGND" H 2000 3880 50  0000 C CNN
-F 2 "" H 2000 3950 60  0000 C CNN
-F 3 "" H 2000 3950 60  0000 C CNN
-	1    2000 3950
 	1    0    0    -1
 $EndComp
@@
 $EndComp
 $Comp
-L FE_V+ #PWR42
+L FE_V+ #PWR038
 U 1 1 526E03BB
 P 6150 2550
-F 0 "#PWR42" H 6150 2650 30  0001 C CNN
+F 0 "#PWR038" H 6150 2650 30  0001 C CNN
 F 1 "FE_V+" H 6150 2650 30  0000 C CNN
 F 2 "~" H 6150 2550 60  0000 C CNN
@@
 	6150 2700 6150 2550
 $Comp
-L GND #PWR45
-U 1 1 526E2673
+L GND_FAN #PWR?
+U 1 1 527CDFF4
+P 8600 1400
+F 0 "#PWR?" H 8600 1400 30  0001 C CNN
+F 1 "GND_FAN" H 8600 1330 30  0000 C CNN
+F 2 "~" H 8600 1400 60  0000 C CNN
+F 3 "~" H 8600 1400 60  0000 C CNN
+	1    8600 1400
+	1    0    0    -1
+$EndComp
+$Comp
+L GND_FAN #PWR?
+U 1 1 527CE004
 P 7900 5550
-F 0 "#PWR45" H 7900 5550 30  0001 C CNN
-F 1 "GND" H 7900 5480 30  0001 C CNN
+F 0 "#PWR?" H 7900 5550 30  0001 C CNN
+F 1 "GND_FAN" H 7900 5480 30  0000 C CNN
 F 2 "~" H 7900 5550 60  0000 C CNN
 F 3 "~" H 7900 5550 60  0000 C CNN
@@
 $EndComp
 $Comp
-L GND #PWR46
-U 1 1 526E268A
-P 8600 1400
-F 0 "#PWR46" H 8600 1400 30  0001 C CNN
-F 1 "GND" H 8600 1330 30  0001 C CNN
-F 2 "~" H 8600 1400 60  0000 C CNN
-F 3 "~" H 8600 1400 60  0000 C CNN
-	1    8600 1400
-	1    0    0    -1
-$EndComp
+L GND_FAN #PWR?
+U 1 1 527CE00A
+P 4700 3750
+F 0 "#PWR?" H 4700 3750 30  0001 C CNN
+F 1 "GND_FAN" H 4700 3680 30  0000 C CNN
+F 2 "~" H 4700 3750 60  0000 C CNN
+F 3 "~" H 4700 3750 60  0000 C CNN
+	1    4700 3750
+	1    0    0    -1
+$EndComp
+$Comp
+L GND_FAN #PWR?
+U 1 1 527CE010
+P 1350 2050
+F 0 "#PWR?" H 1350 2050 30  0001 C CNN
+F 1 "GND_FAN" H 1350 1980 30  0000 C CNN
+F 2 "~" H 1350 2050 60  0000 C CNN
+F 3 "~" H 1350 2050 60  0000 C CNN
+	1    1350 2050
+	1    0    0    -1
+$EndComp
+$Comp
+L GND_FAN #PWR?
+U 1 1 527CE016
+P 2000 3950
+F 0 "#PWR?" H 2000 3950 30  0001 C CNN
+F 1 "GND_FAN" H 2000 3880 30  0000 C CNN
+F 2 "~" H 2000 3950 60  0000 C CNN
+F 3 "~" H 2000 3950 60  0000 C CNN
+	1    2000 3950
+	1    0    0    -1
+$EndComp

Commit message: Layout Work Session 5
Connections:
- net labels added: AGND
- net labels removed: GND_FAN
Changed lines of the file:
@@
-EESchema Schematic File Version 2  date 11/7/2013 10:50:27 PM
+EESchema Schematic File Version 2  date 11/9/2013 9:10:12 PM
 LIBS:power
 LIBS:device
@@
 Sheet 6 9
 Title ""
-Date "8 nov 2013"
+Date "10 nov 2013"
 Rev ""
 Comp ""
@@
 FAN_MODE
 $Comp
-L +12C #PWR034
+L +12C #PWR030
 U 1 1 5243907A
 P 7900 1000
-F 0 "#PWR034" H 7900 970 30  0001 C CNN
+F 0 "#PWR030" H 7900 970 30  0001 C CNN
 F 1 "+12C" H 7900 1110 40  0000 C CNN
 F 2 "~" H 7900 1000 60  0000 C CNN
@@
 	1350 1950 1500 1950
 $Comp
-L +5V #PWR036
+L +5V #PWR031
 U 1 1 525C1500
 P 2000 1700
-F 0 "#PWR036" H 2000 1790 20  0001 C CNN
+F 0 "#PWR031" H 2000 1790 20  0001 C CNN
 F 1 "+5V" H 2000 1790 30  0000 C CNN
 F 2 "~" H 2000 1700 60  0000 C CNN
@@
 $EndComp
 $Comp
-L FE_V+ #PWR038
+L FE_V+ #PWR032
 U 1 1 526E03BB
 P 6150 2550
-F 0 "#PWR038" H 6150 2650 30  0001 C CNN
+F 0 "#PWR032" H 6150 2650 30  0001 C CNN
 F 1 "FE_V+" H 6150 2650 30  0000 C CNN
 F 2 "~" H 6150 2550 60  0000 C CNN
@@
 	6150 2700 6150 2550
 $Comp
-L GND_FAN #PWR?
-U 1 1 527CDFF4
+L AGND #PWR033
+U 1 1 527EEACF
+P 4700 3750
+F 0 "#PWR033" H 4700 3750 40  0001 C CNN
+F 1 "AGND" H 4700 3680 50  0000 C CNN
+F 2 "~" H 4700 3750 60  0000 C CNN
+F 3 "~" H 4700 3750 60  0000 C CNN
+	1    4700 3750
+	1    0    0    -1
+$EndComp
+$Comp
+L AGND #PWR034
+U 1 1 527EEAEB
+P 7900 5550
+F 0 "#PWR034" H 7900 5550 40  0001 C CNN
+F 1 "AGND" H 7900 5480 50  0000 C CNN
+F 2 "~" H 7900 5550 60  0000 C CNN
+F 3 "~" H 7900 5550 60  0000 C CNN
+	1    7900 5550
+	1    0    0    -1
+$EndComp
+$Comp
+L AGND #PWR035
+U 1 1 527EEAF1
+P 2000 3950
+F 0 "#PWR035" H 2000 3950 40  0001 C CNN
+F 1 "AGND" H 2000 3880 50  0000 C CNN
+F 2 "~" H 2000 3950 60  0000 C CNN
+F 3 "~" H 2000 3950 60  0000 C CNN
+	1    2000 3950
+	1    0    0    -1
+$EndComp
+$Comp
+L AGND #PWR036
+U 1 1 527EEAF7
+P 1350 2050
+F 0 "#PWR036" H 1350 2050 40  0001 C CNN
+F 1 "AGND" H 1350 1980 50  0000 C CNN
+F 2 "~" H 1350 2050 60  0000 C CNN
+F 3 "~" H 1350 2050 60  0000 C CNN
+	1    1350 2050
+	1    0    0    -1
+$EndComp
+$Comp
+L AGND #PWR037
+U 1 1 527EEAFD
 P 8600 1400
-F 0 "#PWR?" H 8600 1400 30  0001 C CNN
-F 1 "GND_FAN" H 8600 1330 30  0000 C CNN
+F 0 "#PWR037" H 8600 1400 40  0001 C CNN
+F 1 "AGND" H 8600 1330 50  0000 C CNN
 F 2 "~" H 8600 1400 60  0000 C CNN
 F 3 "~" H 8600 1400 60  0000 C CNN
@@
 	1    0    0    -1
 $EndComp
-$Comp
-L GND_FAN #PWR?
-U 1 1 527CE004
-P 7900 5550
-F 0 "#PWR?" H 7900 5550 30  0001 C CNN
-F 1 "GND_FAN" H 7900 5480 30  0000 C CNN
-F 2 "~" H 7900 5550 60  0000 C CNN
-F 3 "~" H 7900 5550 60  0000 C CNN
-	1    7900 5550
-	1    0    0    -1
-$EndComp
-$Comp
-L GND_FAN #PWR?
-U 1 1 527CE00A
-P 4700 3750
-F 0 "#PWR?" H 4700 3750 30  0001 C CNN
-F 1 "GND_FAN" H 4700 3680 30  0000 C CNN
-F 2 "~" H 4700 3750 60  0000 C CNN
-F 3 "~" H 4700 3750 60  0000 C CNN
-	1    4700 3750
-	1    0    0    -1
-$EndComp
-$Comp
-L GND_FAN #PWR?
-U 1 1 527CE010
-P 1350 2050
-F 0 "#PWR?" H 1350 2050 30  0001 C CNN
-F 1 "GND_FAN" H 1350 1980 30  0000 C CNN
-F 2 "~" H 1350 2050 60  0000 C CNN
-F 3 "~" H 1350 2050 60  0000 C CNN
-	1    1350 2050
-	1    0    0    -1
-$EndComp
-$Comp
-L GND_FAN #PWR?
-U 1 1 527CE016
-P 2000 3950
-F 0 "#PWR?" H 2000 3950 30  0001 C CNN
-F 1 "GND_FAN" H 2000 3880 30  0000 C CNN
-F 2 "~" H 2000 3950 60  0000 C CNN
-F 3 "~" H 2000 3950 60  0000 C CNN
-	1    2000 3950
-	1    0    0    -1
-$EndComp
