File: Power.sch (KiCad schematic (older format))
At the start: 19 parts, among them P1 24 Pin MiniFit JR, SW1 Power Switch

Commit message: Layout Work Session 11 Output
Parts:
- gave numbers to parts that had none: 1
Changed lines of the file:
@@
-EESchema Schematic File Version 2  date 11/13/2013 11:53:23 PM
+EESchema Schematic File Version 2  date 11/17/2013 9:34:47 PM
 LIBS:power
 LIBS:device
@@
 Sheet 9 9
 Title ""
-Date "14 nov 2013"
+Date "18 nov 2013"
 Rev ""
 Comp ""
@@
 $EndComp
 $Comp
-L GND #PWR044
+L GND #PWR50
 U 1 1 523DFA76
 P 1400 1850
-F 0 "#PWR044" H 1400 1850 30  0001 C CNN
+F 0 "#PWR50" H 1400 1850 30  0001 C CNN
 F 1 "GND" H 1400 1780 30  0001 C CNN
 F 2 "" H 1400 1850 60  0000 C CNN
@@
 	5500 1900 5500 1150
 $Comp
-L +12P #PWR045
+L +12P #PWR56
 U 1 1 523DFB91
 P 5500 1150
-F 0 "#PWR045" H 5500 1120 30  0001 C CNN
+F 0 "#PWR56" H 5500 1120 30  0001 C CNN
 F 1 "+12P" H 5500 1250 30  0000 C CNN
 F 2 "" H 5500 1150 60  0000 C CNN
@@
 $EndComp
 $Comp
-L -12P #PWR046
+L -12P #PWR58
 U 1 1 523E04D8
 P 6100 1150
-F 0 "#PWR046" H 6100 1280 20  0001 C CNN
+F 0 "#PWR58" H 6100 1280 20  0001 C CNN
 F 1 "-12P" H 6100 1250 30  0000 C CNN
 F 2 "" H 6100 1150 60  0000 C CNN
@@
 	4800 3200 4800 3450
 $Comp
-L GND #PWR047
+L GND #PWR53
 U 1 1 523E08C4
 P 4800 3450
-F 0 "#PWR047" H 4800 3450 30  0001 C CNN
+F 0 "#PWR53" H 4800 3450 30  0001 C CNN
 F 1 "GND" H 4800 3380 30  0001 C CNN
 F 2 "" H 4800 3450 60  0000 C CNN
@@
 	5650 3000 5650 2750
 $Comp
-L +3.3V #PWR048
+L +3.3V #PWR57
 U 1 1 523E0910
 P 5650 2750
-F 0 "#PWR048" H 5650 2710 30  0001 C CNN
+F 0 "#PWR57" H 5650 2710 30  0001 C CNN
 F 1 "+3.3V" H 5650 2860 30  0000 C CNN
 F 2 "" H 5650 2750 60  0000 C CNN
@@
 $EndComp
 $Comp
-L +12P #PWR049
+L +12P #PWR66
 U 1 1 523E0C76
 P 8000 2250
-F 0 "#PWR049" H 8000 2220 30  0001 C CNN
+F 0 "#PWR66" H 8000 2220 30  0001 C CNN
 F 1 "+12P" H 8000 2350 30  0000 C CNN
 F 2 "" H 8000 2250 60  0000 C CNN
@@
 $EndComp
 $Comp
-L -12P #PWR050
+L -12P #PWR67
 U 1 1 523E0C7C
 P 8000 3800
-F 0 "#PWR050" H 8000 3930 20  0001 C CNN
+F 0 "#PWR67" H 8000 3930 20  0001 C CNN
 F 1 "-12P" H 8000 3900 30  0000 C CNN
 F 2 "" H 8000 3800 60  0000 C CNN
@@
 $EndComp
 $Comp
-L GND #PWR051
+L GND #PWR68
 U 1 1 523E0C82
 P 9000 3200
-F 0 "#PWR051" H 9000 3200 30  0001 C CNN
+F 0 "#PWR68" H 9000 3200 30  0001 C CNN
 F 1 "GND" H 9000 3130 30  0001 C CNN
 F 2 "" H 9000 3200 60  0000 C CNN
@@
 Connection ~ 9450 3050
 $Comp
-L -12V #PWR052
+L -12V #PWR72
 U 1 1 523E0DD3
 P 10350 3800
-F 0 "#PWR052" H 10350 3930 20  0001 C CNN
+F 0 "#PWR72" H 10350 3930 20  0001 C CNN
 F 1 "-12V" H 10350 3900 30  0000 C CNN
 F 2 "" H 10350 3800 60  0000 C CNN
@@
 Connection ~ 9450 2450
 $Comp
-L +12V #PWR053
+L +12V #PWR71
 U 1 1 523E0E37
 P 10350 2200
-F 0 "#PWR053" H 10350 2150 20  0001 C CNN
+F 0 "#PWR71" H 10350 2150 20  0001 C CNN
 F 1 "+12V" H 10350 2300 30  0000 C CNN
 F 2 "" H 10350 2200 60  0000 C CNN
@@
 Connection ~ 3450 1900
 $Comp
-L +12C #PWR054
+L +12C #PWR51
 U 1 1 52438F0D
 P 3450 1150
-F 0 "#PWR054" H 3450 1120 30  0001 C CNN
+F 0 "#PWR51" H 3450 1120 30  0001 C CNN
 F 1 "+12C" H 3450 1260 40  0000 C CNN
 F 2 "~" H 3450 1150 60  0000 C CNN
@@
 $EndComp
 $Comp
-L GND #PWR055
+L GND #PWR69
 U 1 1 524502FC
 P 9400 1650
-F 0 "#PWR055" H 9400 1650 30  0001 C CNN
+F 0 "#PWR69" H 9400 1650 30  0001 C CNN
 F 1 "GND" H 9400 1580 30  0001 C CNN
 F 2 "" H 9400 1650 60  0000 C CNN
@@
 Connection ~ 9400 900
 $Comp
-L +5P #PWR56
+L +5P #PWR55
 U 1 1 52450355
 P 4900 1150
-F 0 "#PWR56" H 4900 1280 20  0001 C CNN
+F 0 "#PWR55" H 4900 1280 20  0001 C CNN
 F 1 "+5P" H 4900 1250 30  0000 C CNN
 F 2 "~" H 4900 1150 60  0000 C CNN
@@
 $EndComp
 $Comp
-L +5V #PWR056
+L +5V #PWR70
 U 1 1 524503B6
 P 10300 650
-F 0 "#PWR056" H 10300 740 20  0001 C CNN
+F 0 "#PWR70" H 10300 740 20  0001 C CNN
 F 1 "+5V" H 10300 740 30  0000 C CNN
 F 2 "~" H 10300 650 60  0000 C CNN
@@
 $EndComp
 $Comp
-L +3.3V #PWR057
+L +3.3V #PWR52
 U 1 1 526E168C
 P 4400 1150
-F 0 "#PWR057" H 4400 1110 30  0001 C CNN
+F 0 "#PWR52" H 4400 1110 30  0001 C CNN
 F 1 "+3.3V" H 4400 1260 30  0000 C CNN
 F 2 "" H 4400 1150 60  0000 C CNN
@@
 $EndComp
 $Comp
-L GND #PWR058
+L GND #PWR59
 U 1 1 527EFE6B
 P 6100 5550
-F 0 "#PWR058" H 6100 5550 30  0001 C CNN
+F 0 "#PWR59" H 6100 5550 30  0001 C CNN
 F 1 "GND" H 6100 5480 30  0001 C CNN
 F 2 "" H 6100 5550 60  0000 C CNN
@@
 $EndComp
 $Comp
-L GND #PWR059
+L GND #PWR54
 U 1 1 52804AA7
 P 4800 7450
-F 0 "#PWR059" H 4800 7450 30  0001 C CNN
+F 0 "#PWR54" H 4800 7450 30  0001 C CNN
 F 1 "GND" H 4800 7380 30  0001 C CNN
 F 2 "" H 4800 7450 60  0000 C CNN
@@
 	5750 6050 6200 6050
 $Comp
-L GND_RELAY #PWR060
+L GND_RELAY #PWR63
 U 1 1 52804C2C
 P 6200 7400
-F 0 "#PWR060" H 6200 7400 30  0001 C CNN
+F 0 "#PWR63" H 6200 7400 30  0001 C CNN
 F 1 "GND_RELAY" H 6200 7330 30  0000 C CNN
 F 2 "~" H 6200 7400 60  0000 C CNN
@@
 $EndComp
 $Comp
-L GND_LED #PWR061
+L GND_LED #PWR62
 U 1 1 52804C3B
 P 6200 6950
-F 0 "#PWR061" H 6200 6950 30  0001 C CNN
+F 0 "#PWR62" H 6200 6950 30  0001 C CNN
 F 1 "GND_LED" H 6200 6880 30  0000 C CNN
 F 2 "~" H 6200 6950 60  0000 C CNN
@@
 $EndComp
 $Comp
-L GND_PWR #PWR062
+L GND_PWR #PWR61
 U 1 1 52804C4A
 P 6200 6550
-F 0 "#PWR062" H 6200 6550 30  0001 C CNN
+F 0 "#PWR61" H 6200 6550 30  0001 C CNN
 F 1 "GND_PWR" H 6200 6480 30  0000 C CNN
 F 2 "~" H 6200 6550 60  0000 C CNN
@@
 $EndComp
 $Comp
-L AGND #PWR063
+L AGND #PWR60
 U 1 1 52804C59
 P 6200 6200
-F 0 "#PWR063" H 6200 6200 40  0001 C CNN
+F 0 "#PWR60" H 6200 6200 40  0001 C CNN
 F 1 "AGND" H 6200 6130 50  0000 C CNN
 F 2 "~" H 6200 6200 60  0000 C CNN
@@
 	6200 7150 5750 7150
 $Comp
-L AGND #PWR064
+L AGND #PWR64
 U 1 1 5284640B
 P 6500 5550
-F 0 "#PWR064" H 6500 5550 40  0001 C CNN
+F 0 "#PWR64" H 6500 5550 40  0001 C CNN
 F 1 "AGND" H 6500 5480 50  0000 C CNN
 F 2 "~" H 6500 5550 60  0000 C CNN
@@
 Connection ~ 6100 5400
 $Comp
-L CONN_1 TP?
+L CONN_1 TP2
 U 1 1 52846001
 P 6400 5250
-F 0 "TP?" H 6480 5250 40  0000 L CNN
+F 0 "TP2" H 6480 5250 40  0000 L CNN
 F 1 "CONN_1" H 6400 5305 30  0001 C CNN
 F 2 "" H 6400 5250 60  0000 C CNN

Commit message: Layout Work Session 12 Output
Parts:
- removed TP2: CONN_1, symbol CONN_1
Connections:
- net AGND: no longer C2.2, C3.2, C4.1, JP1.1, JP2.1, JP3.1, JP4.1, P1.3 (P3), P1.5 (P5), SW1.3, TP1.1
- new net GND: C2.2, C3.2, C4.1, JP1.1, JP2.1, JP3.1, JP4.1, P1.3 (P3), P1.5 (P5), SW1.3, TP1.1
Other:
- moved on the sheet: TP1
Changed lines of the file:
@@
-EESchema Schematic File Version 2  date 11/17/2013 9:34:47 PM
+EESchema Schematic File Version 2  date 11/21/2013 11:46:41 PM
 LIBS:power
 LIBS:device
@@
 Sheet 9 9
 Title ""
-Date "18 nov 2013"
+Date "22 nov 2013"
 Rev ""
 Comp ""
@@
 $EndComp
 $Comp
-L GND #PWR50
+L GND #PWR043
 U 1 1 523DFA76
 P 1400 1850
-F 0 "#PWR50" H 1400 1850 30  0001 C CNN
+F 0 "#PWR043" H 1400 1850 30  0001 C CNN
 F 1 "GND" H 1400 1780 30  0001 C CNN
 F 2 "" H 1400 1850 60  0000 C CNN
@@
 	5500 1900 5500 1150
 $Comp
-L +12P #PWR56
+L +12P #PWR044
 U 1 1 523DFB91
 P 5500 1150
-F 0 "#PWR56" H 5500 1120 30  0001 C CNN
+F 0 "#PWR044" H 5500 1120 30  0001 C CNN
 F 1 "+12P" H 5500 1250 30  0000 C CNN
 F 2 "" H 5500 1150 60  0000 C CNN
@@
 $EndComp
 $Comp
-L -12P #PWR58
+L -12P #PWR045
 U 1 1 523E04D8
 P 6100 1150
-F 0 "#PWR58" H 6100 1280 20  0001 C CNN
+F 0 "#PWR045" H 6100 1280 20  0001 C CNN
 F 1 "-12P" H 6100 1250 30  0000 C CNN
 F 2 "" H 6100 1150 60  0000 C CNN
@@
 	4800 3200 4800 3450
 $Comp
-L GND #PWR53
+L GND #PWR046
 U 1 1 523E08C4
 P 4800 3450
-F 0 "#PWR53" H 4800 3450 30  0001 C CNN
+F 0 "#PWR046" H 4800 3450 30  0001 C CNN
 F 1 "GND" H 4800 3380 30  0001 C CNN
 F 2 "" H 4800 3450 60  0000 C CNN
@@
 	5650 3000 5650 2750
 $Comp
-L +3.3V #PWR57
+L +3.3V #PWR047
 U 1 1 523E0910
 P 5650 2750
-F 0 "#PWR57" H 5650 2710 30  0001 C CNN
+F 0 "#PWR047" H 5650 2710 30  0001 C CNN
 F 1 "+3.3V" H 5650 2860 30  0000 C CNN
 F 2 "" H 5650 2750 60  0000 C CNN
@@
 $EndComp
 $Comp
-L +12P #PWR66
+L +12P #PWR048
 U 1 1 523E0C76
 P 8000 2250
-F 0 "#PWR66" H 8000 2220 30  0001 C CNN
+F 0 "#PWR048" H 8000 2220 30  0001 C CNN
 F 1 "+12P" H 8000 2350 30  0000 C CNN
 F 2 "" H 8000 2250 60  0000 C CNN
@@
 $EndComp
 $Comp
-L -12P #PWR67
+L -12P #PWR049
 U 1 1 523E0C7C
 P 8000 3800
-F 0 "#PWR67" H 8000 3930 20  0001 C CNN
+F 0 "#PWR049" H 8000 3930 20  0001 C CNN
 F 1 "-12P" H 8000 3900 30  0000 C CNN
 F 2 "" H 8000 3800 60  0000 C CNN
@@
 $EndComp
 $Comp
-L GND #PWR68
+L GND #PWR050
 U 1 1 523E0C82
 P 9000 3200
-F 0 "#PWR68" H 9000 3200 30  0001 C CNN
+F 0 "#PWR050" H 9000 3200 30  0001 C CNN
 F 1 "GND" H 9000 3130 30  0001 C CNN
 F 2 "" H 9000 3200 60  0000 C CNN
@@
 Connection ~ 9450 3050
 $Comp
-L -12V #PWR72
+L -12V #PWR051
 U 1 1 523E0DD3
 P 10350 3800
-F 0 "#PWR72" H 10350 3930 20  0001 C CNN
+F 0 "#PWR051" H 10350 3930 20  0001 C CNN
 F 1 "-12V" H 10350 3900 30  0000 C CNN
 F 2 "" H 10350 3800 60  0000 C CNN
@@
 Connection ~ 9450 2450
 $Comp
-L +12V #PWR71
+L +12V #PWR052
 U 1 1 523E0E37
 P 10350 2200
-F 0 "#PWR71" H 10350 2150 20  0001 C CNN
+F 0 "#PWR052" H 10350 2150 20  0001 C CNN
 F 1 "+12V" H 10350 2300 30  0000 C CNN
 F 2 "" H 10350 2200 60  0000 C CNN
@@
 Connection ~ 3450 1900
 $Comp
-L +12C #PWR51
+L +12C #PWR053
 U 1 1 52438F0D
 P 3450 1150
-F 0 "#PWR51" H 3450 1120 30  0001 C CNN
+F 0 "#PWR053" H 3450 1120 30  0001 C CNN
 F 1 "+12C" H 3450 1260 40  0000 C CNN
 F 2 "~" H 3450 1150 60  0000 C CNN
@@
 $EndComp
 $Comp
-L GND #PWR69
+L GND #PWR054
 U 1 1 524502FC
 P 9400 1650
-F 0 "#PWR69" H 9400 1650 30  0001 C CNN
+F 0 "#PWR054" H 9400 1650 30  0001 C CNN
 F 1 "GND" H 9400 1580 30  0001 C CNN
 F 2 "" H 9400 1650 60  0000 C CNN
@@
 $EndComp
 $Comp
-L +5V #PWR70
+L +5V #PWR055
 U 1 1 524503B6
 P 10300 650
-F 0 "#PWR70" H 10300 740 20  0001 C CNN
+F 0 "#PWR055" H 10300 740 20  0001 C CNN
 F 1 "+5V" H 10300 740 30  0000 C CNN
 F 2 "~" H 10300 650 60  0000 C CNN
@@
 $EndComp
 $Comp
-L +3.3V #PWR52
+L +3.3V #PWR056
 U 1 1 526E168C
 P 4400 1150
-F 0 "#PWR52" H 4400 1110 30  0001 C CNN
+F 0 "#PWR056" H 4400 1110 30  0001 C CNN
 F 1 "+3.3V" H 4400 1260 30  0000 C CNN
 F 2 "" H 4400 1150 60  0000 C CNN
@@
 L CONN_1 TP1
 U 1 1 527EFE16
-P 5800 5400
-F 0 "TP1" H 5880 5400 40  0000 L CNN
-F 1 "CONN_1" H 5800 5455 30  0001 C CNN
-F 2 "" H 5800 5400 60  0000 C CNN
-F 3 "" H 5800 5400 60  0000 C CNN
-	1    5800 5400
+P 4650 6050
+F 0 "TP1" H 4730 6050 40  0000 L CNN
+F 1 "CONN_1" H 4650 6105 30  0001 C CNN
+F 2 "" H 4650 6050 60  0000 C CNN
+F 3 "" H 4650 6050 60  0000 C CNN
+	1    4650 6050
 	-1   0    0    1
 $EndComp
-$Comp
-L GND #PWR59
-U 1 1 527EFE6B
-P 6100 5550
-F 0 "#PWR59" H 6100 5550 30  0001 C CNN
-F 1 "GND" H 6100 5480 30  0001 C CNN
-F 2 "" H 6100 5550 60  0000 C CNN
-F 3 "" H 6100 5550 60  0000 C CNN
-	1    6100 5550
-	1    0    0    -1
-$EndComp
-Wire Wire Line
-	6100 5550 6100 5400
-Wire Wire Line
-	5950 5400 6500 5400
-Text Notes 5100 5400 0    60   ~ 0
+Text Notes 4300 6000 0    60   ~ 0
 Star Point
 $Comp
@@
 $EndComp
 $Comp
-L GND #PWR54
+L GND #PWR057
 U 1 1 52804AA7
 P 4800 7450
-F 0 "#PWR54" H 4800 7450 30  0001 C CNN
+F 0 "#PWR057" H 4800 7450 30  0001 C CNN
 F 1 "GND" H 4800 7380 30  0001 C CNN
 F 2 "" H 4800 7450 60  0000 C CNN
@@
 	5750 6050 6200 6050
 $Comp
-L GND_RELAY #PWR63
+L GND_RELAY #PWR058
 U 1 1 52804C2C
 P 6200 7400
-F 0 "#PWR63" H 6200 7400 30  0001 C CNN
+F 0 "#PWR058" H 6200 7400 30  0001 C CNN
 F 1 "GND_RELAY" H 6200 7330 30  0000 C CNN
 F 2 "~" H 6200 7400 60  0000 C CNN
@@
 $EndComp
 $Comp
-L GND_LED #PWR62
+L GND_LED #PWR059
 U 1 1 52804C3B
 P 6200 6950
-F 0 "#PWR62" H 6200 6950 30  0001 C CNN
+F 0 "#PWR059" H 6200 6950 30  0001 C CNN
 F 1 "GND_LED" H 6200 6880 30  0000 C CNN
 F 2 "~" H 6200 6950 60  0000 C CNN
@@
 $EndComp
 $Comp
-L GND_PWR #PWR61
+L GND_PWR #PWR060
 U 1 1 52804C4A
 P 6200 6550
-F 0 "#PWR61" H 6200 6550 30  0001 C CNN
+F 0 "#PWR060" H 6200 6550 30  0001 C CNN
 F 1 "GND_PWR" H 6200 6480 30  0000 C CNN
 F 2 "~" H 6200 6550 60  0000 C CNN
@@
 $EndComp
 $Comp
-L AGND #PWR60
+L AGND #PWR061
 U 1 1 52804C59
 P 6200 6200
-F 0 "#PWR60" H 6200 6200 40  0001 C CNN
+F 0 "#PWR061" H 6200 6200 40  0001 C CNN
 F 1 "AGND" H 6200 6130 50  0000 C CNN
 F 2 "~" H 6200 6200 60  0000 C CNN
@@
 Wire Wire Line
 	6200 7150 5750 7150
-$Comp
-L AGND #PWR64
-U 1 1 5284640B
-P 6500 5550
-F 0 "#PWR64" H 6500 5550 40  0001 C CNN
-F 1 "AGND" H 6500 5480 50  0000 C CNN
-F 2 "~" H 6500 5550 60  0000 C CNN
-F 3 "~" H 6500 5550 60  0000 C CNN
-	1    6500 5550
-	1    0    0    -1
-$EndComp
-Wire Wire Line
-	6500 5400 6500 5550
-Connection ~ 6100 5400
-$Comp
-L CONN_1 TP2
-U 1 1 52846001
-P 6400 5250
-F 0 "TP2" H 6480 5250 40  0000 L CNN
-F 1 "CONN_1" H 6400 5305 30  0001 C CNN
-F 2 "" H 6400 5250 60  0000 C CNN
-F 3 "" H 6400 5250 60  0000 C CNN
-	1    6400 5250
-	0    -1   -1   0
-$EndComp
 $EndSCHEMATC
