File: TerminalBlock.sch (KiCad schematic (older format))
At the start: 2 parts, among them P4 12 Pin Terminal Block, P5 3 Pin TB

Commit message: Layout Work Session 4 Output
Connections:
- net +3.3V: now also P4.10 (P10); no longer P4.6 (P6)
- net +5V: now also P4.9 (P9); no longer P4.7 (P7)
- net FAN_OUT+: now also P4.5 (P5); no longer P4.12 (P12)
- net FAN_OUT-: now also P4.4 (P4); no longer P4.11 (P11)
- net GND: now also P4.8 (P8); no longer P4.3 (P3)
- net TACH_IN: now also P4.3 (P3); no longer P4.10 (P10)
- net TC_IN+: now also P4.7 (P7); no longer P4.8 (P8)
- net TC_IN-: now also P4.6 (P6); no longer P4.9 (P9)
- net V+_ADJ: now also P4.12 (P12); no longer P4.4 (P4)
- net V-_ADJ: now also P4.11 (P11); no longer P4.5 (P5)
Changed lines of the file:
@@
-EESchema Schematic File Version 2  date 11/2/2013 7:04:39 PM
+EESchema Schematic File Version 2  date 11/7/2013 10:50:27 PM
 LIBS:power
 LIBS:device
@@
 Sheet 7 9
 Title ""
-Date "2 nov 2013"
+Date "8 nov 2013"
 Rev ""
 Comp ""
@@
 Comment4 ""
 $EndDescr
-Text HLabel 1925 2000 0    60   Input ~ 0
+Text HLabel 1900 4550 0    60   Input ~ 0
 V+_ADJ
-Text HLabel 1950 2225 0    60   Input ~ 0
+Text HLabel 1900 4400 0    60   Input ~ 0
 V-_ADJ
-Text HLabel 1900 4550 0    60   Output ~ 0
+Text HLabel 1875 2600 0    60   Output ~ 0
 FAN_OUT+
-Text HLabel 1900 4400 0    60   Output ~ 0
+Text HLabel 1875 2325 0    60   Output ~ 0
 FAN_OUT-
-Text HLabel 1850 3750 0    60   Input ~ 0
+Text HLabel 1875 2150 0    60   Input ~ 0
 TACH_IN
 Text HLabel 1450 900  0    60   Output ~ 0
@@
 Text HLabel 1425 1350 0    60   Output ~ 0
 LED_STRING-
-Text HLabel 1850 3350 0    60   Input ~ 0
+Text HLabel 1850 3000 0    60   Input ~ 0
 TC_IN+
-Text HLabel 1850 3600 0    60   Input ~ 0
+Text HLabel 1825 2825 0    60   Input ~ 0
 TC_IN-
 Text HLabel 2850 5500 0    60   BiDi ~ 0
@@
 RELAY_NC
 $Comp
-L +3.3V #PWR47
+L +3.3V #PWR041
 U 1 1 523FFDA7
-P 1075 2250
-F 0 "#PWR47" H 1075 2210 30  0001 C CNN
-F 1 "+3.3V" H 1075 2360 30  0000 C CNN
-F 2 "~" H 1075 2250 60  0000 C CNN
-F 3 "~" H 1075 2250 60  0000 C CNN
-	1    1075 2250
-	1    0    0    -1
-$EndComp
-$Comp
-L +5V #PWR48
+P 750 3500
+F 0 "#PWR041" H 750 3460 30  0001 C CNN
+F 1 "+3.3V" H 750 3610 30  0000 C CNN
+F 2 "~" H 750 3500 60  0000 C CNN
+F 3 "~" H 750 3500 60  0000 C CNN
+	1    750  3500
+	1    0    0    -1
+$EndComp
+$Comp
+L +5V #PWR042
 U 1 1 523FFDB6
-P 1125 2550
-F 0 "#PWR48" H 1125 2640 20  0001 C CNN
-F 1 "+5V" H 1125 2640 30  0000 C CNN
-F 2 "~" H 1125 2550 60  0000 C CNN
-F 3 "~" H 1125 2550 60  0000 C CNN
-	1    1125 2550
+P 1000 3500
+F 0 "#PWR042" H 1000 3590 20  0001 C CNN
+F 1 "+5V" H 1000 3590 30  0000 C CNN
+F 2 "~" H 1000 3500 60  0000 C CNN
+F 3 "~" H 1000 3500 60  0000 C CNN
+	1    1000 3500
 	1    0    0    -1
 $EndComp
@@
 $EndComp
 Wire Wire Line
-	1450 900  5500 900
-Wire Wire Line
 	1425 1350 2050 1350
 Wire Wire Line
@@
 	2200 1100 5500 1100
 Wire Wire Line
-	2200 1100 2200 1750
-Wire Wire Line
-	1800 1750 1800 1800
-Wire Wire Line
-	2350 2000 2350 1200
+	2200 1100 2200 2150
+Wire Wire Line
+	2350 1200 2350 2325
 Wire Wire Line
 	2350 1200 5500 1200
@@
 	5500 1300 2500 1300
 Wire Wire Line
-	2500 1300 2500 2225
-Wire Wire Line
-	2700 2400 2700 1400
+	2500 1300 2500 2600
+Wire Wire Line
+	2700 2825 2700 1400
 Wire Wire Line
 	2700 1400 5500 1400
 Wire Wire Line
-	1850 3350 3000 3350
-Wire Wire Line
-	1850 3600 3200 3600
-Wire Wire Line
-	1850 3750 3400 3750
-Wire Wire Line
-	2850 2550 2850 1500
+	1825 3350 3000 3350
+Wire Wire Line
+	1000 3600 3200 3600
+Wire Wire Line
+	750  3750 3400 3750
+Wire Wire Line
+	2850 1500 2850 3000
 Wire Wire Line
 	2850 1500 5500 1500
@@
 	3250 5800 2850 5800
 Wire Wire Line
-	1125 2550 2850 2550
-Wire Wire Line
-	2700 2400 1075 2400
-Wire Wire Line
-	1075 2400 1075 2250
-Wire Wire Line
-	2500 2225 1950 2225
-Wire Wire Line
-	1925 2000 2350 2000
-$Comp
-L GND #PWR49
-U 1 1 523FFDC5
-P 1800 1800
-F 0 "#PWR49" H 1800 1800 30  0001 C CNN
-F 1 "GND" H 1800 1730 30  0001 C CNN
-F 2 "~" H 1800 1800 60  0000 C CNN
-F 3 "~" H 1800 1800 60  0000 C CNN
-	1    1800 1800
-	1    0    0    -1
-$EndComp
-Wire Wire Line
-	2200 1750 1800 1750
-Wire Wire Line
-	1750 900  1750 900
+	1000 3500 1000 3600
+Wire Wire Line
+	750  3750 750  3500
+Wire Wire Line
+	2850 3000 1850 3000
+Wire Wire Line
+	2350 2325 1875 2325
+Wire Wire Line
+	2500 2600 1875 2600
+Wire Wire Line
+	2200 2150 1875 2150
+Wire Wire Line
+	1825 2825 2700 2825
+$Comp
+L GND #PWR043
+U 1 1 527C695D
+P 1825 3475
+F 0 "#PWR043" H 1825 3475 30  0001 C CNN
+F 1 "GND" H 1825 3405 30  0001 C CNN
+F 2 "~" H 1825 3475 60  0000 C CNN
+F 3 "~" H 1825 3475 60  0000 C CNN
+	1    1825 3475
+	1    0    0    -1
+$EndComp
+Wire Wire Line
+	1825 3475 1825 3350
+Wire Wire Line
+	1450 900  5500 900
 $EndSCHEMATC

Commit message: Layout Work Session 5
Connections:
- net GND renamed GND_PWR
Changed lines of the file:
@@
-EESchema Schematic File Version 2  date 11/7/2013 10:50:27 PM
+EESchema Schematic File Version 2  date 11/9/2013 9:10:12 PM
 LIBS:power
 LIBS:device
@@
 Sheet 7 9
 Title ""
-Date "8 nov 2013"
+Date "10 nov 2013"
 Rev ""
 Comp ""
@@
 RELAY_NC
 $Comp
-L +3.3V #PWR041
+L +3.3V #PWR038
 U 1 1 523FFDA7
 P 750 3500
-F 0 "#PWR041" H 750 3460 30  0001 C CNN
+F 0 "#PWR038" H 750 3460 30  0001 C CNN
 F 1 "+3.3V" H 750 3610 30  0000 C CNN
 F 2 "~" H 750 3500 60  0000 C CNN
@@
 $EndComp
 $Comp
-L +5V #PWR042
+L +5V #PWR039
 U 1 1 523FFDB6
 P 1000 3500
-F 0 "#PWR042" H 1000 3590 20  0001 C CNN
+F 0 "#PWR039" H 1000 3590 20  0001 C CNN
 F 1 "+5V" H 1000 3590 30  0000 C CNN
 F 2 "~" H 1000 3500 60  0000 C CNN
@@
 Wire Wire Line
 	1825 2825 2700 2825
-$Comp
-L GND #PWR043
-U 1 1 527C695D
+Wire Wire Line
+	1825 3475 1825 3350
+Wire Wire Line
+	1450 900  5500 900
+$Comp
+L GND_PWR #PWR040
+U 1 1 527EF77D
 P 1825 3475
-F 0 "#PWR043" H 1825 3475 30  0001 C CNN
-F 1 "GND" H 1825 3405 30  0001 C CNN
+F 0 "#PWR040" H 1825 3475 30  0001 C CNN
+F 1 "GND_PWR" H 1825 3405 30  0000 C CNN
 F 2 "~" H 1825 3475 60  0000 C CNN
 F 3 "~" H 1825 3475 60  0000 C CNN
@@
 	1    0    0    -1
 $EndComp
-Wire Wire Line
-	1825 3475 1825 3350
-Wire Wire Line
-	1450 900  5500 900
 $EndSCHEMATC

Commit message: Layout Work Session 6 Output
Connections:
- net +5V: now also P4.8 (P8); no longer P4.9 (P9)
- net GND_PWR: now also P4.9 (P9); no longer P4.8 (P8)
Changed lines of the file:
@@
-EESchema Schematic File Version 2  date 11/9/2013 9:10:12 PM
+EESchema Schematic File Version 2  date 11/10/2013 9:27:17 PM
 LIBS:power
 LIBS:device
@@
 Sheet 7 9
 Title ""
-Date "10 nov 2013"
+Date "11 nov 2013"
 Rev ""
 Comp ""
@@
 RELAY_NC
 $Comp
-L +3.3V #PWR038
+L +3.3V #PWR44
 U 1 1 523FFDA7
 P 750 3500
-F 0 "#PWR038" H 750 3460 30  0001 C CNN
+F 0 "#PWR44" H 750 3460 30  0001 C CNN
 F 1 "+3.3V" H 750 3610 30  0000 C CNN
 F 2 "~" H 750 3500 60  0000 C CNN
@@
 $EndComp
 $Comp
-L +5V #PWR039
+L +5V #PWR45
 U 1 1 523FFDB6
-P 1000 3500
-F 0 "#PWR039" H 1000 3590 20  0001 C CNN
-F 1 "+5V" H 1000 3590 30  0000 C CNN
-F 2 "~" H 1000 3500 60  0000 C CNN
-F 3 "~" H 1000 3500 60  0000 C CNN
-	1    1000 3500
+P 1800 3200
+F 0 "#PWR45" H 1800 3290 20  0001 C CNN
+F 1 "+5V" H 1800 3290 30  0000 C CNN
+F 2 "~" H 1800 3200 60  0000 C CNN
+F 3 "~" H 1800 3200 60  0000 C CNN
+	1    1800 3200
 	1    0    0    -1
 $EndComp
@@
 	2700 1400 5500 1400
 Wire Wire Line
-	1825 3350 3000 3350
+	1800 3350 3000 3350
 Wire Wire Line
 	1000 3600 3200 3600
 Wire Wire Line
-	750  3750 3400 3750
+	750  4100 3400 4100
 Wire Wire Line
 	2850 1500 2850 3000
@@
 	5500 1800 3400 1800
 Wire Wire Line
-	3400 1800 3400 3750
+	3400 1800 3400 4100
 Wire Wire Line
 	1900 4400 3550 4400
@@
 	3250 5800 2850 5800
 Wire Wire Line
-	1000 3500 1000 3600
-Wire Wire Line
-	750  3750 750  3500
+	750  4100 750  3500
 Wire Wire Line
 	2850 3000 1850 3000
@@
 	1825 2825 2700 2825
 Wire Wire Line
-	1825 3475 1825 3350
-Wire Wire Line
 	1450 900  5500 900
 $Comp
-L GND_PWR #PWR040
+L GND_PWR #PWR46
 U 1 1 527EF77D
-P 1825 3475
-F 0 "#PWR040" H 1825 3475 30  0001 C CNN
-F 1 "GND_PWR" H 1825 3405 30  0000 C CNN
-F 2 "~" H 1825 3475 60  0000 C CNN
-F 3 "~" H 1825 3475 60  0000 C CNN
-	1    1825 3475
-	1    0    0    -1
-$EndComp
+P 1000 3875
+F 0 "#PWR46" H 1000 3875 30  0001 C CNN
+F 1 "GND_PWR" H 1000 3805 30  0000 C CNN
+F 2 "~" H 1000 3875 60  0000 C CNN
+F 3 "~" H 1000 3875 60  0000 C CNN
+	1    1000 3875
+	1    0    0    -1
+$EndComp
+Wire Wire Line
+	1000 3600 1000 3875
+Wire Wire Line
+	1800 3200 1800 3350
 $EndSCHEMATC

Commit message: Layout Work Session 7 Output
Connections:
- net +5V renamed +5P
Changed lines of the file:
@@
-EESchema Schematic File Version 2  date 11/10/2013 9:27:17 PM
+EESchema Schematic File Version 2  date 11/13/2013 1:25:48 AM
 LIBS:power
 LIBS:device
@@
 Sheet 7 9
 Title ""
-Date "11 nov 2013"
+Date "13 nov 2013"
 Rev ""
 Comp ""
@@
 $EndComp
 $Comp
-L +5V #PWR45
-U 1 1 523FFDB6
-P 1800 3200
-F 0 "#PWR45" H 1800 3290 20  0001 C CNN
-F 1 "+5V" H 1800 3290 30  0000 C CNN
-F 2 "~" H 1800 3200 60  0000 C CNN
-F 3 "~" H 1800 3200 60  0000 C CNN
-	1    1800 3200
-	1    0    0    -1
-$EndComp
-$Comp
 L CONN_12 P4
 U 1 1 5258A829
@@
 	1450 900  5500 900
 $Comp
-L GND_PWR #PWR46
+L GND_PWR #PWR45
 U 1 1 527EF77D
 P 1000 3875
-F 0 "#PWR46" H 1000 3875 30  0001 C CNN
+F 0 "#PWR45" H 1000 3875 30  0001 C CNN
 F 1 "GND_PWR" H 1000 3805 30  0000 C CNN
 F 2 "~" H 1000 3875 60  0000 C CNN
@@
 Wire Wire Line
 	1800 3200 1800 3350
+$Comp
+L +5P #PWR46
+U 1 1 52831A41
+P 1800 3200
+F 0 "#PWR46" H 1800 3330 20  0001 C CNN
+F 1 "+5P" H 1800 3300 30  0000 C CNN
+F 2 "~" H 1800 3200 60  0000 C CNN
+F 3 "~" H 1800 3200 60  0000 C CNN
+	1    1800 3200
+	1    0    0    -1
+$EndComp
 $EndSCHEMATC

Commit message: Layout Work Session 11 Output
Connections:
- net TC_IN+: now also P4.6 (P6); no longer P4.7 (P7)
- net TC_IN-: now also P4.7 (P7); no longer P4.6 (P6)
Changed lines of the file:
@@
-EESchema Schematic File Version 2  date 11/13/2013 11:53:23 PM
+EESchema Schematic File Version 2  date 11/17/2013 9:34:47 PM
 LIBS:power
 LIBS:device
@@
 Sheet 7 9
 Title ""
-Date "14 nov 2013"
+Date "18 nov 2013"
 Rev ""
 Comp ""
@@
 Text HLabel 1425 1350 0    60   Output ~ 0
 LED_STRING-
+Text HLabel 1825 2825 0    60   Input ~ 0
+TC_IN+
 Text HLabel 1850 3000 0    60   Input ~ 0
-TC_IN+
-Text HLabel 1825 2825 0    60   Input ~ 0
 TC_IN-
 Text HLabel 2850 5500 0    60   BiDi ~ 0
@@
 RELAY_NC
 $Comp
-L +3.3V #PWR038
+L +3.3V #PWR43
 U 1 1 523FFDA7
 P 750 3500
-F 0 "#PWR038" H 750 3460 30  0001 C CNN
+F 0 "#PWR43" H 750 3460 30  0001 C CNN
 F 1 "+3.3V" H 750 3610 30  0000 C CNN
 F 2 "~" H 750 3500 60  0000 C CNN
@@
 	1450 900  5500 900
 $Comp
-L GND_PWR #PWR039
+L GND_PWR #PWR44
 U 1 1 527EF77D
 P 1000 3875
-F 0 "#PWR039" H 1000 3875 30  0001 C CNN
+F 0 "#PWR44" H 1000 3875 30  0001 C CNN
 F 1 "GND_PWR" H 1000 3805 30  0000 C CNN
 F 2 "~" H 1000 3875 60  0000 C CNN
@@
 	1800 3200 1800 3350
 $Comp
-L +5P #PWR46
+L +5P #PWR45
 U 1 1 52831A41
 P 1800 3200
-F 0 "#PWR46" H 1800 3330 20  0001 C CNN
+F 0 "#PWR45" H 1800 3330 20  0001 C CNN
 F 1 "+5P" H 1800 3300 30  0000 C CNN
 F 2 "~" H 1800 3200 60  0000 C CNN
