File: $Thermocouple.sch (KiCad schematic (older format))
At the start: 25 parts, among them P2 CONN_3X2, P3 CONN_2, U2 MCP3901, U3 LMT84, U4 OPA4170

Commit message: Layout Work Session 14 Output
Connections:
- net AGND: now also C31.1, U2.10 (REFIN-)
Changed lines of the file:
@@
-EESchema Schematic File Version 2  date 11/24/2013 3:13:43 PM
+EESchema Schematic File Version 2  date 11/24/2013 3:26:09 PM
 LIBS:power
 LIBS:device
@@
 Connection ~ 4800 6800
 $Comp
-L +5V #PWR10
+L +5V #PWR01
 U 1 1 5257A1D1
 P 5600 5000
-F 0 "#PWR10" H 5600 5090 20  0001 C CNN
+F 0 "#PWR01" H 5600 5090 20  0001 C CNN
 F 1 "+5V" H 5600 5090 30  0000 C CNN
 F 2 "~" H 5600 5000 60  0000 C CNN
@@
 	6050 3800 6250 3800
 $Comp
-L +5V #PWR11
+L +5V #PWR02
 U 1 1 5257A5A4
 P 5600 5000
-F 0 "#PWR11" H 5600 5090 20  0001 C CNN
+F 0 "#PWR02" H 5600 5090 20  0001 C CNN
 F 1 "+5V" H 5600 5090 30  0000 C CNN
 F 2 "~" H 5600 5000 60  0000 C CNN
@@
 $EndComp
 $Comp
-L +5V #PWR3
+L +5V #PWR03
 U 1 1 5257A5AA
 P 3100 1300
-F 0 "#PWR3" H 3100 1390 20  0001 C CNN
+F 0 "#PWR03" H 3100 1390 20  0001 C CNN
 F 1 "+5V" H 3100 1390 30  0000 C CNN
 F 2 "~" H 3100 1300 60  0000 C CNN
@@
 $EndComp
 $Comp
-L FE_V+ #PWR13
+L FE_V+ #PWR04
 U 1 1 526E01E1
 P 6250 3850
-F 0 "#PWR13" H 6250 3950 30  0001 C CNN
+F 0 "#PWR04" H 6250 3950 30  0001 C CNN
 F 1 "FE_V+" H 6250 3950 30  0000 C CNN
 F 2 "~" H 6250 3850 60  0000 C CNN
@@
 $EndComp
 $Comp
-L FE_V+ #PWR17
+L FE_V+ #PWR05
 U 1 1 526E01F1
 P 9000 5000
-F 0 "#PWR17" H 9000 5100 30  0001 C CNN
+F 0 "#PWR05" H 9000 5100 30  0001 C CNN
 F 1 "FE_V+" H 9000 5100 30  0000 C CNN
 F 2 "~" H 9000 5000 60  0000 C CNN
@@
 $EndComp
 $Comp
-L FE_V+ #PWR14
+L FE_V+ #PWR06
 U 1 1 526E020D
 P 9000 1850
-F 0 "#PWR14" H 9000 1950 30  0001 C CNN
+F 0 "#PWR06" H 9000 1950 30  0001 C CNN
 F 1 "FE_V+" H 9000 1950 30  0000 C CNN
 F 2 "~" H 9000 1850 60  0000 C CNN
@@
 $EndComp
 $Comp
-L AGND #PWR4
+L AGND #PWR07
 U 1 1 527EEF67
 P 3100 4850
-F 0 "#PWR4" H 3100 4850 40  0001 C CNN
+F 0 "#PWR07" H 3100 4850 40  0001 C CNN
 F 1 "AGND" H 3100 4780 50  0000 C CNN
 F 2 "~" H 3100 4850 60  0000 C CNN
@@
 $EndComp
 $Comp
-L AGND #PWR2
+L AGND #PWR08
 U 1 1 527EEF6D
 P 2300 4850
-F 0 "#PWR2" H 2300 4850 40  0001 C CNN
+F 0 "#PWR08" H 2300 4850 40  0001 C CNN
 F 1 "AGND" H 2300 4780 50  0000 C CNN
 F 2 "~" H 2300 4850 60  0000 C CNN
@@
 $EndComp
 $Comp
-L AGND #PWR1
+L AGND #PWR09
 U 1 1 527EEF73
 P 1750 1650
-F 0 "#PWR1" H 1750 1650 40  0001 C CNN
+F 0 "#PWR09" H 1750 1650 40  0001 C CNN
 F 1 "AGND" H 1750 1580 50  0000 C CNN
 F 2 "~" H 1750 1650 60  0000 C CNN
@@
 $EndComp
 $Comp
-L AGND #PWR5
+L AGND #PWR010
 U 1 1 527EEF79
 P 3700 1600
-F 0 "#PWR5" H 3700 1600 40  0001 C CNN
+F 0 "#PWR010" H 3700 1600 40  0001 C CNN
 F 1 "AGND" H 3700 1530 50  0000 C CNN
 F 2 "~" H 3700 1600 60  0000 C CNN
@@
 $EndComp
 $Comp
-L AGND #PWR9
+L AGND #PWR011
 U 1 1 527EEF7F
 P 5600 2800
-F 0 "#PWR9" H 5600 2800 40  0001 C CNN
+F 0 "#PWR011" H 5600 2800 40  0001 C CNN
 F 1 "AGND" H 5600 2730 50  0000 C CNN
 F 2 "~" H 5600 2800 60  0000 C CNN
@@
 $EndComp
 $Comp
-L AGND #PWR8
+L AGND #PWR012
 U 1 1 527EEF85
 P 5550 4000
-F 0 "#PWR8" H 5550 4000 40  0001 C CNN
+F 0 "#PWR012" H 5550 4000 40  0001 C CNN
 F 1 "AGND" H 5550 3930 50  0000 C CNN
 F 2 "~" H 5550 4000 60  0000 C CNN
@@
 $EndComp
 $Comp
-L AGND #PWR7
+L AGND #PWR013
 U 1 1 527EEF8B
 P 4900 4700
-F 0 "#PWR7" H 4900 4700 40  0001 C CNN
+F 0 "#PWR013" H 4900 4700 40  0001 C CNN
 F 1 "AGND" H 4900 4630 50  0000 C CNN
 F 2 "~" H 4900 4700 60  0000 C CNN
@@
 $EndComp
 $Comp
-L AGND #PWR6
+L AGND #PWR014
 U 1 1 527EEF91
 P 4800 6900
-F 0 "#PWR6" H 4800 6900 40  0001 C CNN
+F 0 "#PWR014" H 4800 6900 40  0001 C CNN
 F 1 "AGND" H 4800 6830 50  0000 C CNN
 F 2 "~" H 4800 6900 60  0000 C CNN
@@
 	4450 2200 4450 2450
 Wire Wire Line
-	4450 2600 4450 2900
+	4450 2600 4450 3050
 Wire Wire Line
 	4450 2900 4800 2900
 Wire Wire Line
 	4800 2900 4800 2700
+$Comp
+L AGND #PWR015
+U 1 1 529271FF
+P 4450 3050
+F 0 "#PWR015" H 4450 3050 40  0001 C CNN
+F 1 "AGND" H 4450 2980 50  0000 C CNN
+F 2 "~" H 4450 3050 60  0000 C CNN
+F 3 "~" H 4450 3050 60  0000 C CNN
+	1    4450 3050
+	1    0    0    -1
+$EndComp
+Connection ~ 4450 2900
 $EndSCHEMATC
