File: _autosave-BenchBuddy.kicad_pcb (KiCad board)
At the start: 4 copper layers, 165.1 x 63.5 mm, 140 parts, among them K1 1461069-5, P1 24 Pin MiniFit JR, P2 CONN_3X2, P3 CONN_2, P4 12 Pin Terminal Block, P5 3 Pin TB, Q1 2N3904, Q2 DMN65D8L-7, Q3 AOD476, Q4 AOD476, SW1 Power Switch, U1 LTV-816S, U11 LM317, U2 MCP3901, U3 LMT84, U4 OPA4170, U5 MCP4801, U6 LM337T, U7 AP5726, U8 LM337T, U9 LM317

Commit message: Layout Work Session 14 Output
Parts:
- C30: moved to B.Cu
- moved C30 66.8 mm to (162.9, 104.4), turned to 180 degrees
Routing:
- net N-0000065: track 0.00 -> 3.27 mm, vias 0 -> 1
- net N-0000064: track 0.00 -> 3.12 mm, vias 0 -> 1
- net /Arduino/~RESET: track 47.5 -> 48.9 mm
- net /Arduino/~SHDN: track 36.6 -> 35.7 mm
- net AGND: track 150.0 -> 150.8 mm
- net /Arduino/~LDAC: track 41.3 -> 40.5 mm
- net /Thermocouple/CH1+: track 71.2 -> 71.9 mm
